File: Hardware/PaLampa_MoBo/PaLampa_MoBo_H00/LED_Drivers.kicad_sch (KiCad schematic)
At the start: 13 parts

Commit message: HW updates
Parts:
- gave numbers to parts that had none: 13
Changed lines of the file:
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@@
   (symbol (lib_id "power:GND") (at 148.59 134.62 0) (unit 1)
     (in_bom yes) (on_board yes) (fields_autoplaced)
-    (property "Reference" "#PWR?" (id 0) (at 148.59 140.97 0)
+    (property "Reference" "#PWR0112" (id 0) (at 148.59 140.97 0)
       (effects (font (size 1.27 1.27)) hide)
     )
@@
   (symbol (lib_id "power:GND") (at 88.9 134.62 0) (unit 1)
     (in_bom yes) (on_board yes) (fields_autoplaced)
-    (property "Reference" "#PWR?" (id 0) (at 88.9 140.97 0)
+    (property "Reference" "#PWR0119" (id 0) (at 88.9 140.97 0)
       (effects (font (size 1.27 1.27)) hide)
     )
@@
   (symbol (lib_id "Device:L") (at 124.46 66.04 90) (unit 1)
     (in_bom yes) (on_board yes) (fields_autoplaced)
-    (property "Reference" "L?" (id 0) (at 124.46 61.8322 90))
+    (property "Reference" "L1" (id 0) (at 124.46 61.8322 90))
     (property "Value" "6u8" (id 1) (at 124.46 64.3691 90))
     (property "Footprint" "PaLampa_Library:L_Cenker_CKCS5040" (id 2) (at 124.46 66.04 0)
@@
   (symbol (lib_id "Device:D_Schottky") (at 135.89 109.22 180) (unit 1)
     (in_bom yes) (on_board yes) (fields_autoplaced)
-    (property "Reference" "D?" (id 0) (at 136.2075 104.2502 0))
+    (property "Reference" "D6" (id 0) (at 136.2075 104.2502 0))
     (property "Value" "SS54" (id 1) (at 136.2075 106.7871 0))
     (property "Footprint" "Diode_SMD:D_SMA" (id 2) (at 135.89 109.22 0)
@@
   (symbol (lib_id "Device:D_Schottky") (at 135.89 66.04 180) (unit 1)
     (in_bom yes) (on_board yes) (fields_autoplaced)
-    (property "Reference" "D?" (id 0) (at 136.2075 61.0702 0))
+    (property "Reference" "D5" (id 0) (at 136.2075 61.0702 0))
     (property "Value" "SS54" (id 1) (at 136.2075 63.6071 0))
     (property "Footprint" "Diode_SMD:D_SMA" (id 2) (at 135.89 66.04 0)
@@
   (symbol (lib_id "power:GND") (at 166.37 134.62 0) (unit 1)
     (in_bom yes) (on_board yes) (fields_autoplaced)
-    (property "Reference" "#PWR?" (id 0) (at 166.37 140.97 0)
+    (property "Reference" "#PWR0111" (id 0) (at 166.37 140.97 0)
       (effects (font (size 1.27 1.27)) hide)
     )
@@
   (symbol (lib_id "Device:C") (at 166.37 123.19 0) (unit 1)
     (in_bom yes) (on_board yes) (fields_autoplaced)
-    (property "Reference" "C?" (id 0) (at 169.291 122.3553 0)
+    (property "Reference" "C20" (id 0) (at 169.291 122.3553 0)
       (effects (font (size 1.27 1.27)) (justify left))
     )
@@
   (symbol (lib_id "Device:C") (at 166.37 80.01 0) (unit 1)
     (in_bom yes) (on_board yes) (fields_autoplaced)
-    (property "Reference" "C?" (id 0) (at 169.291 79.1753 0)
+    (property "Reference" "C10" (id 0) (at 169.291 79.1753 0)
       (effects (font (size 1.27 1.27)) (justify left))
     )
@@
   (symbol (lib_id "Connector_Generic:Conn_02x04_Odd_Even") (at 232.41 88.9 0) (unit 1)
     (in_bom yes) (on_board yes) (fields_autoplaced)
-    (property "Reference" "J?" (id 0) (at 233.68 81.3902 0))
+    (property "Reference" "J2" (id 0) (at 233.68 81.3902 0))
     (property "Value" "Conn_02x04_Odd_Even" (id 1) (at 233.68 83.9271 0))
     (property "Footprint" "Connector_IDC:IDC-Header_2x04_P2.54mm_Vertical" (id 2) (at 232.41 88.9 0)
@@
   (symbol (lib_id "power:GND") (at 116.84 134.62 0) (unit 1)
     (in_bom yes) (on_board yes) (fields_autoplaced)
-    (property "Reference" "#PWR?" (id 0) (at 116.84 140.97 0)
+    (property "Reference" "#PWR0120" (id 0) (at 116.84 140.97 0)
       (effects (font (size 1.27 1.27)) hide)
     )
@@
   (symbol (lib_id "Device:L") (at 124.46 109.22 90) (unit 1)
     (in_bom yes) (on_board yes) (fields_autoplaced)
-    (property "Reference" "L?" (id 0) (at 124.46 105.0122 90))
+    (property "Reference" "L2" (id 0) (at 124.46 105.0122 90))
     (property "Value" "6u8" (id 1) (at 124.46 107.5491 90))
     (property "Footprint" "PaLampa_Library:L_Cenker_CKCS5040" (id 2) (at 124.46 109.22 0)
@@
   (symbol (lib_id "power:GND") (at 148.59 91.44 0) (unit 1)
     (in_bom yes) (on_board yes) (fields_autoplaced)
-    (property "Reference" "#PWR?" (id 0) (at 148.59 97.79 0)
+    (property "Reference" "#PWR0122" (id 0) (at 148.59 97.79 0)
       (effects (font (size 1.27 1.27)) hide)
     )
@@
   (symbol (lib_id "PaLampa_Library:SY7203") (at 124.46 123.19 0) (unit 1)
     (in_bom yes) (on_board yes) (fields_autoplaced)
-    (property "Reference" "U?" (id 0) (at 124.46 111.9242 0))
+    (property "Reference" "U7" (id 0) (at 124.46 111.9242 0))
     (property "Value" "SY7203" (id 1) (at 124.46 114.4611 0))
     (property "Footprint" "PaLampa_Library:DFN-10-1EP_3x3mm_P0.5mm_EP1.75x2.6mm" (id 2) (at 125.095 116.84 0)
@@
   (symbol (lib_id "Device:C") (at 88.9 123.19 0) (unit 1)
     (in_bom yes) (on_board yes) (fields_autoplaced)
-    (property "Reference" "C?" (id 0) (at 91.821 122.3553 0)
+    (property "Reference" "C9" (id 0) (at 91.821 122.3553 0)
       (effects (font (size 1.27 1.27)) (justify left))
     )
@@
   (symbol (lib_id "power:GND") (at 166.37 91.44 0) (unit 1)
     (in_bom yes) (on_board yes) (fields_autoplaced)
-    (property "Reference" "#PWR?" (id 0) (at 166.37 97.79 0)
+    (property "Reference" "#PWR0121" (id 0) (at 166.37 97.79 0)
       (effects (font (size 1.27 1.27)) hide)
     )
@@
   (symbol (lib_id "PaLampa_Library:SY7203") (at 124.46 80.01 0) (unit 1)
     (in_bom yes) (on_board yes) (fields_autoplaced)
-    (property "Reference" "U?" (id 0) (at 124.46 68.7442 0))
+    (property "Reference" "U6" (id 0) (at 124.46 68.7442 0))
     (property "Value" "SY7203" (id 1) (at 124.46 71.2811 0))
     (property "Footprint" "PaLampa_Library:DFN-10-1EP_3x3mm_P0.5mm_EP1.75x2.6mm" (id 2) (at 125.095 73.66 0)
@@
   (symbol (lib_id "power:GND") (at 88.9 91.44 0) (unit 1)
     (in_bom yes) (on_board yes) (fields_autoplaced)
-    (property "Reference" "#PWR?" (id 0) (at 88.9 97.79 0)
+    (property "Reference" "#PWR0114" (id 0) (at 88.9 97.79 0)
       (effects (font (size 1.27 1.27)) hide)
     )
@@
   (symbol (lib_id "Device:R") (at 148.59 87.63 0) (unit 1)
     (in_bom yes) (on_board yes)
-    (property "Reference" "R?" (id 0) (at 150.368 86.7953 0)
+    (property "Reference" "R4" (id 0) (at 150.368 86.7953 0)
       (effects (font (size 1.27 1.27)) (justify left))
     )
@@
   (symbol (lib_id "Device:R") (at 148.59 130.81 0) (unit 1)
     (in_bom yes) (on_board yes)
-    (property "Reference" "R?" (id 0) (at 150.368 129.9753 0)
+    (property "Reference" "R5" (id 0) (at 150.368 129.9753 0)
       (effects (font (size 1.27 1.27)) (justify left))
     )
@@
   (symbol (lib_id "power:GND") (at 116.84 91.44 0) (unit 1)
     (in_bom yes) (on_board yes) (fields_autoplaced)
-    (property "Reference" "#PWR?" (id 0) (at 116.84 97.79 0)
+    (property "Reference" "#PWR0117" (id 0) (at 116.84 97.79 0)
       (effects (font (size 1.27 1.27)) hide)
     )
@@
   (symbol (lib_id "power:GND") (at 209.55 95.25 0) (unit 1)
     (in_bom yes) (on_board yes) (fields_autoplaced)
-    (property "Reference" "#PWR?" (id 0) (at 209.55 101.6 0)
+    (property "Reference" "#PWR0126" (id 0) (at 209.55 101.6 0)
       (effects (font (size 1.27 1.27)) hide)
     )
@@
   (symbol (lib_id "power:+5V") (at 262.89 82.55 0) (unit 1)
     (in_bom yes) (on_board yes) (fields_autoplaced)
-    (property "Reference" "#PWR?" (id 0) (at 262.89 86.36 0)
+    (property "Reference" "#PWR0127" (id 0) (at 262.89 86.36 0)
       (effects (font (size 1.27 1.27)) hide)
     )
@@
   (symbol (lib_id "power:+5V") (at 88.9 109.22 0) (unit 1)
     (in_bom yes) (on_board yes) (fields_autoplaced)
-    (property "Reference" "#PWR?" (id 0) (at 88.9 113.03 0)
+    (property "Reference" "#PWR0118" (id 0) (at 88.9 113.03 0)
       (effects (font (size 1.27 1.27)) hide)
     )
@@
   (symbol (lib_id "Device:C") (at 88.9 80.01 0) (unit 1)
     (in_bom yes) (on_board yes) (fields_autoplaced)
-    (property "Reference" "C?" (id 0) (at 91.821 79.1753 0)
+    (property "Reference" "C8" (id 0) (at 91.821 79.1753 0)
       (effects (font (size 1.27 1.27)) (justify left))
     )
@@
   (symbol (lib_id "power:+5V") (at 88.9 66.04 0) (unit 1)
     (in_bom yes) (on_board yes) (fields_autoplaced)
-    (property "Reference" "#PWR?" (id 0) (at 88.9 69.85 0)
-      (effects (font (size 1.27 1.27)) hide)
-    )
+    (property "Reference" "#PWR0113" (id 0) (at 88.9 69.85 0)
+      (effects (font (size 1.27 1.27)) hide)
+    )
