File: Hardware/PaLampa_MoBo/PaLampa_MoBo_H00/PaLampa_MoBo_H00.kicad_pcb (KiCad board)
At the start: 2 copper layers, 83 parts, among them J1 Conn_01x03_Male, J2 Conn_02x04_Odd_Even, J7 918-418K2023S40001, J9 Conn_01x05_Male, Q1 2N7002, Q2 S8050, Q3 S8050, Q4 2N7002, SW1 SW_SPST, SW2 SW_SPST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

Commit message: HW updates
Parts:
- removed TP+5V1, TPGND1: TestPoint, Connector_Wire:SolderWirePad_1x01_SMD_1x2mm
- moved C21 251.9 mm to (1.68, 13.4), turned to -90 degrees
- moved C22 248.2 mm to (3.71, 15.1), turned to -90 degrees
- moved U8 244.4 mm to (4.67, 11.7)
- moved C16 237.9 mm to (14.8, 12.6), turned to 90 degrees
- moved R8 237.3 mm to (18.0, 12.6), turned to -90 degrees
- moved R9 236.3 mm to (16.4, 12.6), turned to -90 degrees
- moved C11 236.0 mm to (25.3, 4.78), turned to 90 degrees
- moved D4 235.2 mm to (21.2, 3.91), turned to 90 degrees
- moved R10 233.7 mm to (18.7, 24.4), turned to 180 degrees
- moved J7 232.3 mm to (13.7, 3.20), turned to 180 degrees
- moved Q2 230.5 mm to (20.7, 27.1)
- moved C14 229.1 mm to (28.1, 27.7), turned to -90 degrees
- moved C13 229.0 mm to (20.4, 20.3), turned to 90 degrees
- moved U5 228.1 mm to (14.2, 18.3), turned to -90 degrees
- moved Q3 227.2 mm to (16.7, 27.1), turned to 180 degrees
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Connections:
- net Net-(J7-PadA7) renamed /USB+Power/D-
- U1 pad 10: /LED_Drivers/COLD_PWM -> BUTTON2
- U1 pad 11: /LED_Drivers/WARM_PWM -> BUTTON3
- U1 pad 16: /USB+Power/FUSB_INT -> BUZZER
- U1 pad 28: BUZZER -> unconnected-(U1-Pad28)
- U1 pad 29: BUTTON3 -> /LED_Drivers/WARM_PWM
- U1 pad 30: BUTTON1 -> /LED_Drivers/COLD_PWM
- U1 pad 31: BUTTON2 -> /USB+Power/FUSB_INT
- U1 pad 9: unconnected-(U1-Pad9) -> BUTTON1
Routing:
- net +5V: track 0.00 -> 52.0 mm
- net /LED_Drivers/WARM_PWM: track 0.00 -> 27.1 mm, vias 0 -> 2
- net GND: track 0.00 -> 25.0 mm, vias 0 -> 12
- net WARM_ANODE: track 0.00 -> 21.6 mm
- net +3V3: track 0.00 -> 21.1 mm
- net /LED_Drivers/WS2812_DATA: track 0.00 -> 18.9 mm, vias 0 -> 2
- net /LED_Drivers/COLD_PWM: track 0.00 -> 16.4 mm, vias 0 -> 4
- net COLD_ANODE: track 0.00 -> 16.0 mm
- net COLD_CATHODE: track 0.00 -> 14.5 mm, vias 0 -> 1
- net /USB+Power/D-: track 0.00 -> 12.0 mm, vias 0 -> 2
- net /USB+Power/D+: track 0.00 -> 11.9 mm
- net WARM_CATHODE: track 0.00 -> 10.6 mm
- net Net-(J7-PadA5): track 0.00 -> 9.74 mm, vias 0 -> 2
- net Net-(J7-PadB5): track 0.00 -> 3.49 mm
- net Net-(R8-Pad2): track 0.00 -> 2.67 mm
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- added copper zone on F.Cu, net +5V
- added copper zone on F.Cu, net COLD_ANODE
- added copper zone on F.Cu, net Net-(D5-Pad2)
- added copper zone on F.Cu, net Net-(D6-Pad2)
- added copper zone on F.Cu, net WARM_ANODE
Other:
- board outline added: 60 x 100 mm
