File: Hardware/PaLampa_MoBo/PaLampa_MoBo_H00/PaLampa_MoBo_H00.kicad_pcb (KiCad board)
At the start: 2 copper layers, 60 x 100 mm, 81 parts, among them J1 Conn_01x03_Male, J2 Conn_02x04_Odd_Even, J7 918-418K2023S40001, J9 Conn_01x05_Male, Q1 2N7002, Q2 S8050, Q3 S8050, Q4 2N7002, SW1 SW_SPST, SW2 SW_SPST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

Commit message: Completed H00 revision. Added production data.
Parts:
- removed H5, H6: MountingHole, MountingHole:MountingHole_3.2mm_M3
- added G4: CoufalElektronika_logo, PaLampa_Library:Coufal_elektronika_notext_10mm, F.Cu at (30.0, 56.0)
- G1, G2, G5, U2: moved to B.Cu
- moved G5 193.6 mm to (3.68, 43.2), turned to -90 degrees
- moved R14 190.9 mm to (9.81, 97.0)
- moved H3 190.8 mm to (4.00, 96.0)
- moved R22 176.8 mm to (11.0, 92.7)
- moved J1 166.8 mm to (20.6, 54.5), turned to -90 degrees
- moved C17 150.3 mm to (10.8, 89.2)
- moved R15 147.1 mm to (9.02, 90.9), turned to 180 degrees
- moved R13 145.7 mm to (56.5, 27.1), turned to 180 degrees
- moved R2 141.6 mm to (36.8, 45.7), turned to 90 degrees
- moved R21 141.3 mm to (56.5, 28.8), turned to 180 degrees
- moved U2 140.3 mm to (51.3, 64.9), turned to 180 degrees
- moved C7 136.7 mm to (50.0, 67.9)
- moved R18 134.9 mm to (31.2, 69.0), turned to 90 degrees
- moved G2 133.4 mm to (26.5, 25.7), turned to 180 degrees
- moved C3 132.2 mm to (25.1, 45.7), turned to 90 degrees
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Connections:
- net /LED_Drivers/COLD_PWM renamed /COLD_PWM
- net /LED_Drivers/WARM_PWM renamed /WARM_PWM
- net Net-(Q4-Pad2) renamed /WS2812_3V3
Routing:
- net +3V3: track 21.1 -> 258.2 mm, vias 0 -> 2
- net I2C_SCL: track 0.00 -> 101.2 mm, vias 0 -> 4
- net I2C_SDA: track 0.00 -> 98.2 mm, vias 0 -> 5
- net +5V: track 52.0 -> 145.4 mm, vias 0 -> 3
- net LIGHT1: track 0.00 -> 78.5 mm, vias 0 -> 4
- net /USB+Power/ESP_RST: track 0.00 -> 77.3 mm, vias 0 -> 2
- net BUTTON3: track 0.00 -> 63.6 mm, vias 0 -> 2
- net BUZZER: track 0.00 -> 59.7 mm, vias 0 -> 2
- net BUTTON2: track 0.00 -> 57.2 mm, vias 0 -> 2
- net GND: track 25.0 -> 80.2 mm, vias 12 -> 27
- net BUTTON1: track 0.00 -> 53.7 mm, vias 0 -> 2
- net /WARM_PWM: track 27.1 -> 80.0 mm, vias 2 -> 4
- net TEMPERATURE: track 0.00 -> 52.1 mm, vias 0 -> 2
- net /COLD_PWM: track 16.4 -> 67.3 mm, vias 4 -> 6
- net LIGHT2: track 0.00 -> 47.2 mm, vias 0 -> 2
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- added copper zone on B.Cu, net GND
Other:
- board text added: "GND SCL SDA 3V3 5V0"
- board text added: "PaLampa project by the Vedatori team. Electronics designed by Marek Coufal."
- board text added: "PaLampa_MoBo_H00 04-2023"
