File: Hardware/PaLampa_MoBo/PaLampa_MoBo_H00/PaLampa_MoBo_H00.kicad_sch (KiCad schematic)
At the start: 48 parts, among them J9 Conn_01x05_Male, Q1 2N7002, Q4 2N7002, SW1 SW_SPST, SW2 SW_SPST, SW3 SW_SPST, U1 ESP32-WROOM-32D, U2 DS18B20

Commit message: HW updates
Parts:
- BZ1: footprint Time-O-Mat_Library:Buzzer_12x9.5RM6.6 -> PaLampa_Library:Buzzer_12x9.5RM6.6
- G1: footprint Time-O-Mat_Library:Coufal_elektronika_text_30x13mm -> PaLampa_Library:Coufal_elektronika_text_30x13mm
- G2, G3: footprint Time-O-Mat_Library:Vedatori_15mm -> PaLampa_Library:Vedatori_15mm
- G5: footprint Time-O-Mat_Library:Espressif_logo_30mm -> PaLampa_Library:Espressif_logo_30mm; now left out of the parts list
- H1, H2, H3, H4, H5, H6: now left out of the parts list
- R12: footprint Connector_JST:JST_XH_S2B-XH-A-1_1x02_P2.50mm_Horizontal -> OptoDevice:R_LDR_5.1x4.3mm_P3.4mm_Vertical
- gave numbers to parts that had none: 3
Connections:
- net BUTTON1: now also U1.9 (IO33); no longer U1.30 (IO18)
- net BUTTON2: now also U1.10 (IO25); no longer U1.31 (IO19)
- net BUTTON3: now also U1.11 (IO26); no longer U1.29 (IO5)
- net BUZZER: now also U1.16 (IO13); no longer U1.28 (IO17)
- net LED_Drivers/COLD_PWM: now also U1.30 (IO18); no longer U1.10 (IO25)
- net LED_Drivers/WARM_PWM: now also U1.29 (IO5); no longer U1.11 (IO26)
- net USB+Power/FUSB_INT: now also U1.31 (IO19); no longer U1.16 (IO13)
- no-connect marks 9 -> 6
