File: Hardware/PaLampa_MoBo/PaLampa_MoBo_H00/PaLampa_MoBo_H00.kicad_sch (KiCad schematic)
At the start: 48 parts, among them J1 Conn_01x03_Male, J9 Conn_01x05_Male, Q1 2N7002, Q4 2N7002, SW1 SW_SPST, SW2 SW_SPST, SW3 SW_SPST, U1 ESP32-WROOM-32D, U2 DS18B20, U3 OLED_I2C

Commit message: Completed H00 revision. Added production data.
Parts:
- removed H5, H6: MountingHole, MountingHole:MountingHole_3.2mm_M3, symbol Mechanical:MountingHole
- added G4: CoufalElektronika_logo, PaLampa_Library:Coufal_elektronika_notext_10mm, symbol Time-O-Mat_Library:CoufalElektronika_logo
- G1, G2, G3: now left out of the parts list
Connections:
- net WS2812_3V3: now reaches Q4.2 (S), R16.2, U1.27 (IO16)
- net LED_Drivers/COLD_PWM renamed COLD_PWM
- net LED_Drivers/WARM_PWM renamed WARM_PWM
Changed lines of the file:
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@@
     (stroke (width 0) (type default))
   )
-  (wire (pts (xy 139.7 49.53) (xy 139.7 82.55))
+  (wire (pts (xy 144.78 49.53) (xy 144.78 82.55))
     (stroke (width 0) (type default))
   )
@@
     (stroke (width 0) (type default))
   )
-  (wire (pts (xy 114.3 49.53) (xy 139.7 49.53))
+  (wire (pts (xy 114.3 49.53) (xy 144.78 49.53))
     (stroke (width 0) (type default))
   )
@@
     (stroke (width 0) (type default))
   )
-  (wire (pts (xy 139.7 82.55) (xy 229.87 82.55))
+  (wire (pts (xy 144.78 82.55) (xy 229.87 82.55))
     (stroke (width 0) (type default))
   )
@@
   (text "• MTDI/GPIO12: internal pull-down\n• GPIO0: internal pull-up\n• GPIO2: internal pull-down\n• GPIO4: internal pull-down\n• MTDO/GPIO15: internal pull-up\n• GPIO5: internal pull-up"
     (at 45.72 62.23 0)
+    (effects (font (size 1.27 1.27)) (justify left bottom))
+  )
+  (label "WARM_PWM" (at 130.81 49.53 0) (fields_autoplaced)
+    (effects (font (size 1.27 1.27)) (justify left bottom))
+  )
+  (label "WS2812_3V3" (at 130.81 62.23 0) (fields_autoplaced)
+    (effects (font (size 1.27 1.27)) (justify left bottom))
+  )
+  (label "COLD_PWM" (at 130.81 67.31 0) (fields_autoplaced)
     (effects (font (size 1.27 1.27)) (justify left bottom))
   )
@@
   )
   (symbol (lib_id "Time-O-Mat_Library:Vedatori_logo") (at 251.46 173.99 0) (unit 1)
-    (in_bom yes) (on_board yes) (dnp no) (fields_autoplaced)
+    (in_bom no) (on_board yes) (dnp no) (fields_autoplaced)
     (property "Reference" "G2" (at 251.46 170.627 0)
       (effects (font (size 1.27 1.27)) hide)
@@
     )
   )
-  (symbol (lib_id "Mechanical:MountingHole") (at 45.72 36.83 0) (unit 1)
-    (in_bom no) (on_board yes) (dnp no)
-    (property "Reference" "H5" (at 48.26 35.6616 0)
-      (effects (font (size 1.27 1.27)) (justify left))
-    )
-    (property "Value" "MountingHole" (at 48.26 37.973 0)
-      (effects (font (size 1.27 1.27)) (justify left))
-    )
-    (property "Footprint" "MountingHole:MountingHole_3.2mm_M3" (at 45.72 36.83 0)
-      (effects (font (size 1.27 1.27)) hide)
-    )
-    (property "Datasheet" "~" (at 45.72 36.83 0)
-      (effects (font (size 1.27 1.27)) hide)
-    )
-    (instances
-      (project "PaLampa_MoBo_H00"
-        (path "/68867493-9f89-4388-916e-56f5ada0ac5c"
-          (reference "H5") (unit 1)
-        )
-      )
-    )
-  )
   (symbol (lib_id "Device:D_Schottky") (at 67.31 83.82 270) (unit 1)
     (in_bom yes) (on_board yes) (dnp no)
@@
         (path "/68867493-9f89-4388-916e-56f5ada0ac5c"
           (reference "#PWR0133") (unit 1)
-        )
-      )
-    )
-  )
-  (symbol (lib_id "Mechanical:MountingHole") (at 45.72 41.91 0) (unit 1)
-    (in_bom no) (on_board yes) (dnp no)
-    (property "Reference" "H6" (at 48.26 40.7416 0)
-      (effects (font (size 1.27 1.27)) (justify left))
-    )
-    (property "Value" "MountingHole" (at 48.26 43.053 0)
-      (effects (font (size 1.27 1.27)) (justify left))
-    )
-    (property "Footprint" "MountingHole:MountingHole_3.2mm_M3" (at 45.72 41.91 0)
-      (effects (font (size 1.27 1.27)) hide)
-    )
-    (property "Datasheet" "~" (at 45.72 41.91 0)
-      (effects (font (size 1.27 1.27)) hide)
-    )
-    (instances
-      (project "PaLampa_MoBo_H00"
-        (path "/68867493-9f89-4388-916e-56f5ada0ac5c"
-          (reference "H6") (unit 1)
         )
       )
@@
     )
   )
+  (symbol (lib_id "Time-O-Mat_Library:CoufalElektronika_logo") (at 264.16 157.48 0) (unit 1)
+    (in_bom no) (on_board yes) (dnp no) (fields_autoplaced)
+    (property "Reference" "G4" (at 264.16 150.6188 0)
+      (effects (font (size 1.27 1.27)) hide)
+    )
+    (property "Value" "CoufalElektronika_logo" (at 264.16 164.3412 0)
+      (effects (font (size 1.27 1.27)) hide)
+    )
+    (property "Footprint" "PaLampa_Library:Coufal_elektronika_notext_10mm" (at 264.16 157.48 0)
+      (effects (font (size 1.27 1.27)) hide)
+    )
+    (property "Datasheet" "" (at 264.16 157.48 0)
+      (effects (font (size 1.27 1.27)) hide)
+    )
+    (instances
+      (project "PaLampa_MoBo_H00"
+        (path "/68867493-9f89-4388-916e-56f5ada0ac5c"
+          (reference "G4") (unit 1)
+        )
+      )
+    )
+  )
   (symbol (lib_id "Device:D_Schottky") (at 55.88 173.99 270) (unit 1)
     (in_bom yes) (on_board yes) (dnp no)
@@
   )
   (symbol (lib_id "Time-O-Mat_Library:Vedatori_logo") (at 270.51 173.99 0) (unit 1)
-    (in_bom yes) (on_board yes) (dnp no) (fields_autoplaced)
+    (in_bom no) (on_board yes) (dnp no) (fields_autoplaced)
     (property "Reference" "G3" (at 270.51 170.627 0)
       (effects (font (size 1.27 1.27)) hide)
@@
   )
   (symbol (lib_id "Time-O-Mat_Library:CoufalElektronika_logo") (at 223.52 173.99 0) (unit 1)
-    (in_bom yes) (on_board yes) (dnp no) (fields_autoplaced)
+    (in_bom no) (on_board yes) (dnp no) (fields_autoplaced)
     (property "Reference" "G1" (at 223.52 167.1288 0)
       (effects (font (size 1.27 1.27)) hide)
