File: Hardware/PaLampa_MoBo/PaLampa_MoBo_H00/USB+Power.kicad_sch (KiCad schematic)
At the start: 20 parts, among them J7 918-418K2023S40001, Q2 S8050, Q3 S8050, U4 AMS1117-3.3, U5 CH340G, U8 FUSB302BMPX

Commit message: changed electrolytic capacitor part number
Parts:
- C11, C19: LCSC C43803 -> C43348
Changed lines of the file:
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@@
       (effects (font (size 1.27 1.27)) hide)
     )
-    (property "LCSC" "C43803" (at 152.4 132.08 0)
+    (property "LCSC" "C43348" (at 152.4 132.08 0)
       (effects (font (size 1.27 1.27)) hide)
     )
@@
       (effects (font (size 1.27 1.27)) hide)
     )
-    (property "LCSC" "C43803" (at 34.29 73.66 0)
+    (property "LCSC" "C43348" (at 34.29 73.66 0)
       (effects (font (size 1.27 1.27)) hide)
     )
