File: Hardware/PaLampa_LED/PaLampa_LED_H00/PaLampa_LED_H00.kicad_pcb (KiCad board)
At the start: 2 copper layers, 59 x 73 mm, 74 parts, among them J1 Conn_02x04_Odd_Even

Commit message: Completed H00 revision. Added production data.
Changed lines of the file:
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@@
     (fp_line (start 13.28 5.1) (end 13.28 -12.72)
       (stroke (width 0.1) (type solid)) (layer "B.Fab"))
-    (pad "1" thru_hole roundrect (at 0 0 90) (size 1.7 1.7) (drill 1) (layers "*.Cu" "*.Mask") (roundrect_rratio 0.147059)
+    (pad "1" thru_hole roundrect (at 0 0 90) (size 1.7 1.7) (drill 1) (layers "*.Cu" "*.Mask") (roundrect_rratio 0.1470588235)
       (net 67 "WARM_ANODE") (pinfunction "Pin_1") (pintype "passive"))
     (pad "2" thru_hole circle (at 2.54 0 90) (size 1.7 1.7) (drill 1) (layers "*.Cu" "*.Mask")
