File: Hardware/PaLampa_LED/PaLampa_LED_H01/PaLampa_LED_H01.kicad_pcb (KiCad board)
At the start: 2 copper layers, 59 x 73 mm, 74 parts, among them J1 Conn_02x04_Odd_Even

Commit message: H01 changes
Parts:
- added J2: Conn_01x03, Connector_JST:JST_XH_S3B-XH-A_1x03_P2.50mm_Horizontal, B.Cu at (52.8, 38.9)
- added R2: R, Resistor_SMD:R_0402_1005Metric, F.Cu at (2.67, 36.8)
- added U1: DS18B20, Package_TO_SOT_THT:TO-92_Inline, B.Cu at (4.50, 35.0)
- G1: footprint PaLampa_Library:Coufal_elektronika_text_30x13mm -> PaLampa_Library:Coufal_elektronika_notext_10mm
- G2: footprint PaLampa_Library:Vedatori_15mm -> PaLampa_Library:VedatoriNew_40x5,7mm
- moved G2 13.9 mm to (17.5, 36.5), turned to -90 degrees
- moved G1 6.49 mm to (29.5, 36.5), turned to -90 degrees
- moved R1 2.27 mm to (22.0, 67.8)
Connections:
- J1 pad 5: GND -> Net-(J1-Pin_5)
- WS16 pad 2: unconnected-(WS16-Pad2) -> Net-(J2-Pin_1)
Routing:
- net Net-(J1-Pin_5): track 0.00 -> 58.7 mm
- net Net-(J2-Pin_1): track 0.00 -> 40.6 mm, vias 0 -> 2
- net +5V: track 0.00 -> 22.4 mm, vias 0 -> 3
- net GND: track 45.2 -> 65.1 mm, vias 34 -> 35
- net Net-(WS1-DIN): track 6.29 -> 3.71 mm
- net WS_DATA: track 5.53 -> 6.10 mm, vias 0 -> 2
Other:
- outline, holes or cut-outs redrawn
- board text added: "PCB designed by Marek Coufal"
- board text added: "PaLampa_LED_H01 06-2023"
