File: Hardware/PaLampa_LED/PaLampa_LED_H01/PaLampa_LED_H01.kicad_sch (KiCad schematic)
At the start: 74 parts, among them J1 Conn_02x04_Odd_Even

Commit message: H01 changes
Parts:
- added J2: Conn_01x03, Connector_JST:JST_XH_S3B-XH-A_1x03_P2.50mm_Horizontal, symbol Connector_Generic:Conn_01x03
- added R2: 4K7, Resistor_SMD:R_0402_1005Metric, symbol Device:R
- added U1: DS18B20, Package_TO_SOT_THT:TO-92_Inline, symbol Sensor_Temperature:DS18B20
- G1: footprint PaLampa_Library:Coufal_elektronika_text_30x13mm -> PaLampa_Library:Coufal_elektronika_notext_10mm
- G2: footprint PaLampa_Library:Vedatori_15mm -> PaLampa_Library:VedatoriNew_40x5,7mm
Connections:
- net +5V: now also J2.2 (Pin_2), R2.1, U1.3 (V_{DD})
- net GND: now also J2.3 (Pin_3), U1.1 (GND); no longer J1.5 (Pin_5)
- net at WS16.2 (DOUT): now also J2.1 (Pin_1)
- new net: J1.5 (Pin_5), R2.2, U1.2 (DQ)
- no-connect marks 1 -> 0
