File: Hardware/PaLampa_MoBo/PaLampa_MoBo_H01/LED_Drivers.kicad_sch (KiCad schematic)
At the start: 13 parts, among them J2 Conn_02x04_Odd_Even, U6 SY7203, U7 SY7203

Commit message: H01 changes
Connections:
- net GND: no longer J2.5 (Pin_5)
- new net LED_TEMP: J2.5 (Pin_5)
Changed lines of the file:
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@@
   (junction (at 116.84 109.22) (diameter 0) (color 0 0 0 0)
   )
-  (junction (at 227.33 90.17) (diameter 0) (color 0 0 0 0)
-  )
   (junction (at 132.08 109.22) (diameter 0) (color 0 0 0 0)
   )
@@
     (stroke (width 0) (type default))
   )
+  (wire (pts (xy 207.01 91.44) (xy 227.33 91.44))
+    (stroke (width 0) (type default))
+  )
   (wire (pts (xy 88.9 66.04) (xy 116.84 66.04))
     (stroke (width 0) (type default))
@@
     (stroke (width 0) (type default))
   )
-  (wire (pts (xy 209.55 90.17) (xy 209.55 95.25))
+  (wire (pts (xy 209.55 88.9) (xy 209.55 95.25))
     (stroke (width 0) (type default))
   )
@@
     (stroke (width 0) (type default))
   )
-  (wire (pts (xy 227.33 90.17) (xy 227.33 88.9))
-    (stroke (width 0) (type default))
-  )
   (wire (pts (xy 116.84 66.04) (xy 116.84 76.2))
     (stroke (width 0) (type default))
@@
     (stroke (width 0) (type default))
   )
-  (wire (pts (xy 227.33 91.44) (xy 227.33 90.17))
-    (stroke (width 0) (type default))
-  )
   (wire (pts (xy 132.08 119.38) (xy 132.08 109.22))
     (stroke (width 0) (type default))
@@
     (stroke (width 0) (type default))
   )
-  (wire (pts (xy 227.33 90.17) (xy 209.55 90.17))
+  (wire (pts (xy 227.33 88.9) (xy 209.55 88.9))
     (stroke (width 0) (type default))
   )
@@
     (effects (font (size 1.27 1.27)) (justify right))
   )
+  (hierarchical_label "LED_TEMP" (shape bidirectional) (at 207.01 91.44 180) (fields_autoplaced)
+    (effects (font (size 1.27 1.27)) (justify right))
+  )
   (hierarchical_label "WS2812_DATA" (shape input) (at 240.03 91.44 0) (fields_autoplaced)
     (effects (font (size 1.27 1.27)) (justify left))
@@
     (pin "1")
     (instances
-      (project "PaLampa_MoBo_H00"
+      (project "PaLampa_MoBo_H01"
         (path "/68867493-9f89-4388-916e-56f5ada0ac5c/4ac9ab7b-b59d-4d9f-a955-f58805b17013"
           (reference "#PWR0112") (unit 1)
@@
     (pin "1")
     (instances
-      (project "PaLampa_MoBo_H00"
+      (project "PaLampa_MoBo_H01"
         (path "/68867493-9f89-4388-916e-56f5ada0ac5c/4ac9ab7b-b59d-4d9f-a955-f58805b17013"
           (reference "#PWR0119") (unit 1)
@@
     (pin "2")
     (instances
-      (project "PaLampa_MoBo_H00"
+      (project "PaLampa_MoBo_H01"
         (path "/68867493-9f89-4388-916e-56f5ada0ac5c/4ac9ab7b-b59d-4d9f-a955-f58805b17013"
           (reference "L1") (unit 1)
@@
     (pin "2")
     (instances
-      (project "PaLampa_MoBo_H00"
+      (project "PaLampa_MoBo_H01"
         (path "/68867493-9f89-4388-916e-56f5ada0ac5c/4ac9ab7b-b59d-4d9f-a955-f58805b17013"
           (reference "D6") (unit 1)
@@
     (pin "2")
     (instances
-      (project "PaLampa_MoBo_H00"
+      (project "PaLampa_MoBo_H01"
         (path "/68867493-9f89-4388-916e-56f5ada0ac5c/4ac9ab7b-b59d-4d9f-a955-f58805b17013"
           (reference "D5") (unit 1)
@@
     (pin "1")
     (instances
-      (project "PaLampa_MoBo_H00"
+      (project "PaLampa_MoBo_H01"
         (path "/68867493-9f89-4388-916e-56f5ada0ac5c/4ac9ab7b-b59d-4d9f-a955-f58805b17013"
           (reference "#PWR0111") (unit 1)
@@
     (pin "2")
     (instances
-      (project "PaLampa_MoBo_H00"
+      (project "PaLampa_MoBo_H01"
         (path "/68867493-9f89-4388-916e-56f5ada0ac5c/4ac9ab7b-b59d-4d9f-a955-f58805b17013"
           (reference "C20") (unit 1)
@@
     (pin "2")
     (instances
-      (project "PaLampa_MoBo_H00"
+      (project "PaLampa_MoBo_H01"
         (path "/68867493-9f89-4388-916e-56f5ada0ac5c/4ac9ab7b-b59d-4d9f-a955-f58805b17013"
           (reference "C10") (unit 1)
@@
     (pin "8")
     (instances
-      (project "PaLampa_MoBo_H00"
+      (project "PaLampa_MoBo_H01"
         (path "/68867493-9f89-4388-916e-56f5ada0ac5c/4ac9ab7b-b59d-4d9f-a955-f58805b17013"
           (reference "J2") (unit 1)
@@
     (pin "1")
     (instances
-      (project "PaLampa_MoBo_H00"
+      (project "PaLampa_MoBo_H01"
         (path "/68867493-9f89-4388-916e-56f5ada0ac5c/4ac9ab7b-b59d-4d9f-a955-f58805b17013"
           (reference "#PWR0120") (unit 1)
@@
     (pin "2")
     (instances
-      (project "PaLampa_MoBo_H00"
+      (project "PaLampa_MoBo_H01"
         (path "/68867493-9f89-4388-916e-56f5ada0ac5c/4ac9ab7b-b59d-4d9f-a955-f58805b17013"
           (reference "L2") (unit 1)
@@
     (pin "1")
     (instances
-      (project "PaLampa_MoBo_H00"
+      (project "PaLampa_MoBo_H01"
         (path "/68867493-9f89-4388-916e-56f5ada0ac5c/4ac9ab7b-b59d-4d9f-a955-f58805b17013"
           (reference "#PWR0122") (unit 1)
@@
     (pin "9")
     (instances
-      (project "PaLampa_MoBo_H00"
+      (project "PaLampa_MoBo_H01"
         (path "/68867493-9f89-4388-916e-56f5ada0ac5c/4ac9ab7b-b59d-4d9f-a955-f58805b17013"
           (reference "U7") (unit 1)
@@
     (pin "2")
     (instances
-      (project "PaLampa_MoBo_H00"
+      (project "PaLampa_MoBo_H01"
         (path "/68867493-9f89-4388-916e-56f5ada0ac5c/4ac9ab7b-b59d-4d9f-a955-f58805b17013"
           (reference "C9") (unit 1)
@@
     (pin "1")
     (instances
-      (project "PaLampa_MoBo_H00"
+      (project "PaLampa_MoBo_H01"
         (path "/68867493-9f89-4388-916e-56f5ada0ac5c/4ac9ab7b-b59d-4d9f-a955-f58805b17013"
           (reference "#PWR0121") (unit 1)
@@
     (pin "9")
     (instances
-      (project "PaLampa_MoBo_H00"
+      (project "PaLampa_MoBo_H01"
         (path "/68867493-9f89-4388-916e-56f5ada0ac5c/4ac9ab7b-b59d-4d9f-a955-f58805b17013"
           (reference "U6") (unit 1)
@@
     (pin "1")
     (instances
-      (project "PaLampa_MoBo_H00"
+      (project "PaLampa_MoBo_H01"
         (path "/68867493-9f89-4388-916e-56f5ada0ac5c/4ac9ab7b-b59d-4d9f-a955-f58805b17013"
           (reference "#PWR0114") (unit 1)
@@
     (pin "2")
     (instances
-      (project "PaLampa_MoBo_H00"
+      (project "PaLampa_MoBo_H01"
         (path "/68867493-9f89-4388-916e-56f5ada0ac5c/4ac9ab7b-b59d-4d9f-a955-f58805b17013"
           (reference "R4") (unit 1)
@@
     (pin "2")
     (instances
-      (project "PaLampa_MoBo_H00"
+      (project "PaLampa_MoBo_H01"
         (path "/68867493-9f89-4388-916e-56f5ada0ac5c/4ac9ab7b-b59d-4d9f-a955-f58805b17013"
           (reference "R5") (unit 1)
@@
     (pin "1")
     (instances
-      (project "PaLampa_MoBo_H00"
+      (project "PaLampa_MoBo_H01"
         (path "/68867493-9f89-4388-916e-56f5ada0ac5c/4ac9ab7b-b59d-4d9f-a955-f58805b17013"
           (reference "#PWR0117") (unit 1)
@@
     (pin "1")
     (instances
-      (project "PaLampa_MoBo_H00"
+      (project "PaLampa_MoBo_H01"
         (path "/68867493-9f89-4388-916e-56f5ada0ac5c/4ac9ab7b-b59d-4d9f-a955-f58805b17013"
           (reference "#PWR0126") (unit 1)
@@
     (pin "1")
     (instances
-      (project "PaLampa_MoBo_H00"
+      (project "PaLampa_MoBo_H01"
         (path "/68867493-9f89-4388-916e-56f5ada0ac5c/4ac9ab7b-b59d-4d9f-a955-f58805b17013"
           (reference "#PWR0127") (unit 1)
@@
     (pin "1")
     (instances
-      (project "PaLampa_MoBo_H00"
+      (project "PaLampa_MoBo_H01"
         (path "/68867493-9f89-4388-916e-56f5ada0ac5c/4ac9ab7b-b59d-4d9f-a955-f58805b17013"
           (reference "#PWR0118") (unit 1)
@@
     (pin "2")
     (instances
-      (project "PaLampa_MoBo_H00"
+      (project "PaLampa_MoBo_H01"
         (path "/68867493-9f89-4388-916e-56f5ada0ac5c/4ac9ab7b-b59d-4d9f-a955-f58805b17013"
           (reference "C8") (unit 1)
@@
     (pin "1")
     (instances
-      (project "PaLampa_MoBo_H00"
+      (project "PaLampa_MoBo_H01"
         (path "/68867493-9f89-4388-916e-56f5ada0ac5c/4ac9ab7b-b59d-4d9f-a955-f58805b17013"
           (reference "#PWR0113") (unit 1)

Commit message: H01 update
Parts:
- R4, R5: footprint Resistor_SMD:R_0603_1608Metric -> Resistor_SMD:R_1206_3216Metric; LCSC C175664 -> C175854
Changed lines of the file:
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@@
       (effects (font (size 1.27 1.27)) (justify left))
     )
-    (property "Footprint" "Resistor_SMD:R_0603_1608Metric" (at 146.812 87.63 90)
+    (property "Footprint" "Resistor_SMD:R_1206_3216Metric" (at 146.812 87.63 90)
       (effects (font (size 1.27 1.27)) hide)
     )
@@
       (effects (font (size 1.27 1.27)) hide)
     )
-    (property "LCSC" "C175664" (at 148.59 87.63 0)
+    (property "LCSC" "C175854" (at 148.59 87.63 0)
       (effects (font (size 1.27 1.27)) hide)
     )
@@
       (effects (font (size 1.27 1.27)) (justify left))
     )
-    (property "Footprint" "Resistor_SMD:R_0603_1608Metric" (at 146.812 130.81 90)
+    (property "Footprint" "Resistor_SMD:R_1206_3216Metric" (at 146.812 130.81 90)
       (effects (font (size 1.27 1.27)) hide)
     )
@@
       (effects (font (size 1.27 1.27)) hide)
     )
-    (property "LCSC" "C175664" (at 148.59 130.81 0)
+    (property "LCSC" "C175854" (at 148.59 130.81 0)
       (effects (font (size 1.27 1.27)) hide)
     )
