File: Hardware/PaLampa_MoBo/PaLampa_MoBo_H01/PaLampa_MoBo_H01.kicad_pcb (KiCad board)
At the start: 2 copper layers, 60 x 100 mm, 80 parts, among them J1 Conn_01x03_Male, J2 Conn_02x04_Odd_Even, J7 918-418K2023S40001, J9 Conn_01x05_Male, Q1 2N7002, Q2 S8050, Q3 S8050, Q4 2N7002, SW1 SW_SPST, SW2 SW_SPST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

Commit message: H01 changes
Parts:
- G2, G3: footprint PaLampa_Library:Vedatori_15mm -> PaLampa_Library:VedatoriNew_40x5,7mm
- U3: footprint PaLampa_Library:Display_128x64_096_I2C -> PaLampa_Library:Display_128x64_096_I2C_3Hole
- moved BZ1 11.7 mm to (40.9, 86.5)

Commit message: H01 update
Parts:
- removed G3: Vedatori_logo, PaLampa_Library:VedatoriNew_40x5,7mm
- removed J1: Conn_01x03_Male, Connector_PinHeader_2.54mm:PinHeader_1x03_P2.54mm_Vertical
- added J3: Conn_01x02, Connector_JST:JST_XH_B2B-XH-A_1x02_P2.50mm_Vertical, F.Cu at (17.9, 55.9)
- added Q5: 2N7002, Package_TO_SOT_SMD:SOT-23, F.Cu at (47.9, 23.1)
- added R6: 10K, Resistor_SMD:R_0603_1608Metric, F.Cu at (50.8, 23.0)
- added R7: 10K, Resistor_SMD:R_0603_1608Metric, F.Cu at (39.1, 11.2)
- R12: moved to B.Cu
- R4, R5: footprint Resistor_SMD:R_0603_1608Metric -> Resistor_SMD:R_1206_3216Metric
- moved R14 42.7 mm to (29.9, 59.3), turned to 90 degrees
- moved R12 42.7 mm to (29.2, 2.54), turned to 180 degrees
- moved G4 35.6 mm to (54.2, 30.0)
- moved R13 34.0 mm to (29.7, 6.15)
- moved R21 34.0 mm to (29.7, 7.92)
- moved C15 33.7 mm to (27.2, 6.96)
- moved R15 24.9 mm to (24.5, 71.4)
- moved R22 24.9 mm to (26.4, 73.2)
- moved C17 24.9 mm to (26.2, 69.6)
- moved C11 6.37 mm to (22.7, 10.6), turned to 180 degrees
- moved R4 0.67 mm to (49.4, 11.5)
- moved R5 0.55 mm to (30.2, 11.5)
Connections:
- J2 pad 5: GND -> /LED_Drivers/LED_TEMP
- U1 pad 12: TOUCH7 -> unconnected-(U1-IO27-Pad12)
- U1 pad 28: unconnected-(U1-IO17-Pad28) -> /COLD_PWM
- U1 pad 30: /COLD_PWM -> /LED_TEMP_3V3
Routing:
- net LIGHT1: track 78.5 -> 136.3 mm
- net +3V3: track 258.2 -> 301.2 mm, vias 2 -> 4
- net /LED_TEMP_3V3: track 0.00 -> 29.3 mm, vias 0 -> 2
- net /LED_Drivers/LED_TEMP: track 0.00 -> 27.3 mm, vias 0 -> 2
- net Net-(R14-Pad2): track 7.49 -> 27.5 mm, vias 0 -> 2
- net +5V: track 145.4 -> 158.3 mm
- net Net-(BZ1-+): track 13.3 -> 25.1 mm
- net GND: track 80.2 -> 74.9 mm
- net TOUCH7: track 4.19 -> 0.00 mm
- net Net-(R12-Pad2): track 4.47 -> 8.31 mm
- net LIGHT2: track 47.2 -> 44.8 mm, vias 2 -> 4
- net I2C_SCL: track 101.2 -> 103.3 mm
- net I2C_SDA: track 98.2 -> 100.2 mm
- net TEMPERATURE: track 52.1 -> 54.1 mm
- net BUZZER: track 59.7 -> 61.7 mm
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Other:
- board text added: "Do NOT disconnect LEDs when powered on! Neodpojujte LEDky když je deska zapnutá!"

Commit message: H01 updates
Routing:
- net /LED_TEMP_3V3: track 29.3 -> 65.2 mm
- net GND: track 74.9 -> 76.6 mm, vias 27 -> 28
- net /COLD_PWM: track 65.8 -> 67.1 mm
Other:
- board text added: "PaLampa_MoBo_H01 06-2023"
- board text removed: "PaLampa_MoBo_H00 04-2023"
